File: PCB/v1/bot/bot.sch (EAGLE design)
At the start: 3 parts, among them J1 SMA-J-P-H-ST-EM1

Commit message: updates
Parts:
- removed PAD1: (no value), wirepad:2,54/0,8
- added PAD2: (no value), wirepad:2,54/1,1
Connections:
- net GND: now also PAD2.P; no longer PAD1.P
Changed lines of the file:
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@@
 <?xml version="1.0" encoding="utf-8"?>
 <!DOCTYPE eagle SYSTEM "eagle.dtd">
-<eagle version="9.3.0">
+<eagle version="9.3.2">
 <drawing>
 <settings>
@@
 <parts>
 <part name="J1" library="SMA-J-P-H-ST-EM1" deviceset="SMA-J-P-H-ST-EM1" device=""/>
-<part name="PAD1" library="wirepad" library_urn="urn:adsk.eagle:library:412" deviceset="2,54/0,8" device="" package3d_urn="urn:adsk.eagle:package:30838/1"/>
 <part name="U$1" library="new_inductor" deviceset="INDUCTOR" device=""/>
+<part name="PAD2" library="wirepad" library_urn="urn:adsk.eagle:library:412" deviceset="2,54/1,1" device="" package3d_urn="urn:adsk.eagle:package:30836/1"/>
 </parts>
 <sheets>
@@
 <attribute name="VALUE" x="-55.880659375" y="22.859009375" size="1.78166875" layer="96"/>
 </instance>
-<instance part="PAD1" gate="P" x="-5.08" y="22.86" smashed="yes" rot="MR0">
-<attribute name="NAME" x="-3.937" y="24.7142" size="1.778" layer="95" rot="MR0"/>
-<attribute name="VALUE" x="-3.937" y="19.558" size="1.778" layer="96" rot="MR0"/>
-</instance>
 <instance part="U$1" gate="G$1" x="-35.56" y="30.48" smashed="yes">
 <attribute name="VALUE" x="-37.5412" y="26.2128" size="3.4798" layer="96" ratio="10" rot="SR0"/>
 <attribute name="NAME" x="-36.4744" y="33.8328" size="3.4798" layer="95" ratio="10" rot="SR0"/>
+</instance>
+<instance part="PAD2" gate="1" x="-5.08" y="17.78" smashed="yes" rot="R90">
+<attribute name="NAME" x="-6.9342" y="16.637" size="1.778" layer="95" rot="R90"/>
+<attribute name="VALUE" x="-1.778" y="16.637" size="1.778" layer="96" rot="R90"/>
 </instance>
 </instances>
@@
 <segment>
 <pinref part="J1" gate="G$1" pin="GND"/>
-<pinref part="PAD1" gate="P" pin="P"/>
 <wire x1="-40.64" y1="27.94" x2="-40.64" y2="22.86" width="0.1524" layer="91"/>
-<wire x1="-40.64" y1="22.86" x2="-7.62" y2="22.86" width="0.1524" layer="91"/>
+<wire x1="-40.64" y1="22.86" x2="-5.08" y2="22.86" width="0.1524" layer="91"/>
+<pinref part="PAD2" gate="1" pin="P"/>
+<wire x1="-5.08" y1="22.86" x2="-5.08" y2="20.32" width="0.1524" layer="91"/>
 </segment>
 </net>
