File: PCB/v1/top/top.brd (EAGLE design)
At the start: 19.9 x 32.1 mm, 1 part

Commit message: updates
Parts:
- moved PAD1 12.8 mm to (24.6, 20.5)
Routing:
- net N$1: track 5.80 -> 7.08 mm
Changed lines of the file:
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@@
 <?xml version="1.0" encoding="utf-8"?>
 <!DOCTYPE eagle SYSTEM "eagle.dtd">
-<eagle version="9.3.0">
+<eagle version="9.3.2">
 <drawing>
 <settings>
@@
 <wire x1="27.9" y1="31.6" x2="8" y2="31.6" width="0" layer="20"/>
 <wire x1="8" y1="31.6" x2="8" y2="-0.5" width="0" layer="20"/>
-<rectangle x1="16.2" y1="0" x2="20.2" y2="31" layer="1" rot="R180"/>
-<hole x="12" y="26" drill="4.5"/>
-<hole x="12" y="6" drill="4.5"/>
-<hole x="24" y="26" drill="4.5"/>
+<rectangle x1="16.2" y1="0.2" x2="20.2" y2="31.2" layer="1" rot="R180"/>
+<hole x="12" y="27.5" drill="3"/>
+<hole x="12" y="3.5" drill="3"/>
+<hole x="24" y="27.5" drill="3"/>
 <dimension x1="8" y1="31.6" x2="8" y2="-0.5" x3="2" y3="15.55" textsize="1.778" layer="255"/>
-<hole x="24" y="6" drill="4.5"/>
+<hole x="24" y="3.5" drill="3"/>
 </plain>
 <attributes>
@@
 </autorouter>
 <elements>
-<element name="PAD1" library="wirepad" library_urn="urn:adsk.eagle:library:412" package="2,54/0,8" package3d_urn="urn:adsk.eagle:package:30838/1" value="" x="11.8" y="20.5" smashed="yes">
-<attribute name="NAME" x="10.53" y="22.024" size="1.27" layer="25" ratio="10"/>
-<attribute name="VALUE" x="11.8" y="21.1" size="0.0254" layer="27"/>
+<element name="PAD1" library="wirepad" library_urn="urn:adsk.eagle:library:412" package="2,54/0,8" package3d_urn="urn:adsk.eagle:package:30838/1" value="" x="24.6" y="20.5" smashed="yes">
+<attribute name="NAME" x="23.33" y="22.024" size="1.27" layer="25" ratio="10"/>
+<attribute name="VALUE" x="24.6" y="21.1" size="0.0254" layer="27"/>
 </element>
 </elements>
@@
 <signal name="N$1">
 <contactref element="PAD1" pad="1"/>
-<wire x1="17.6" y1="20.5" x2="11.8" y2="20.5" width="0.8128" layer="1"/>
+<wire x1="24.4" y1="20.7" x2="24.6" y2="20.5" width="0.8128" layer="1"/>
+<wire x1="24.4" y1="20.7" x2="17.6" y2="20.7" width="0.8128" layer="1"/>
 </signal>
 </signals>
